Commit message: Rover description update

File: description/robot1.urdf.xacro (robot description, xacro)
@@ -11,7 +11,7 @@
     <!-- <xacro:include filename="vectornav_imu.xacro"/> -->
     <xacro:include filename="robot1_zed_camera.xacro"/>
-    <xacro:if value="$(arg use_lidar)">
+    <!-- <xacro:if value="$(arg use_lidar)">
         <xacro:include filename="lidar.xacro"/>
-    </xacro:if>
+    </xacro:if> -->
     <!-- Build robot model -->
     <xacro:robot_description prefix="$(arg prefix)" camera_name="$(arg camera_name)" camera_model="$(arg camera_model)"/>

File: description/robot33333_core.xacro (robot description, xacro)
@@ -1,5 +1,5 @@
 <?xml version="1.0"?>
 <robot xmlns:xacro="http://www.ros.org/wiki/xacro">
-    <xacro:macro name="robot_description" params="prefix camera_name=zedm camera_model=zedm">
+  <xacro:macro name="robot_description" params="prefix camera_name=zedm camera_model=zedm">
     <!-- Properties -->
     <xacro:if value="${prefix != ''}">
@@ -48,5 +48,9 @@
             filename="file://$(find arcs_cohort_description)/meshes/robot1_base_link.STL" />
         </geometry>
-        <material name="red"/>
+        <material
+          name="">
+          <color
+            rgba="0.792156862745098 0.819607843137255 0.933333333333333 1" />
+        </material>
       </visual>
       <collision>
@@ -60,18 +64,19 @@
       </collision>
     </link>
-    <link name="${prefix_}front_left_wheel_link">
-      <inertial>
-          <origin
-            xyz="-1.888E-07 3.5593E-07 0.0069273"
-            rpy="0 0 0" />
-          <mass
-            value="0.13821" />
-          <inertia
-            ixx="0.0003215"
-            ixy="4.0549E-10"
-            ixz="-2.1303E-10"
-            iyy="0.0003215"
-            iyz="-1.0165E-10"
-            izz="0.00063022" />
+    <link
+      name="${prefix_}front_left_wheel_link">
+      <inertial>
+        <origin
+          xyz="-1.888E-07 3.5593E-07 0.0069273"
+          rpy="0 0 0" />
+        <mass
+          value="0.13821" />
+        <inertia
+          ixx="0.0003215"
+          ixy="4.0549E-10"
+          ixz="-2.1303E-10"
+          iyy="0.0003215"
+          iyz="-1.0165E-10"
+          izz="0.00063022" />
       </inertial>
       <visual>
@@ -83,5 +88,9 @@
             filename="file://$(find arcs_cohort_description)/meshes/robot1_front_left_wheel_link.STL" />
         </geometry>
-        <material name="yellow"/>
+        <material
+          name="">
+          <color
+            rgba="0.79216 0.81961 0.93333 1" />
+        </material>
       </visual>
       <collision>
@@ -100,5 +109,5 @@
       <origin
         xyz="0.108 0.089 0.01825"
-        rpy="-1.57 0 0" />
+        rpy="-1.5708 0 0" />
       <parent
         link="${prefix_}base_link" />
@@ -108,21 +117,22 @@
         xyz="0 0 1" />
       <dynamics
-        damping="1000000.0"
+        damping="0"
         friction="0" />
     </joint>
-    <link name="${prefix_}front_right_wheel_link">
-      <inertial>
-          <origin
-            xyz="-1.888E-07 3.5593E-07 0.0069273"
-            rpy="0 0 0" />
-          <mass
-            value="0.13821" />
-          <inertia
-            ixx="0.0003215"
-            ixy="4.0549E-10"
-            ixz="-2.1303E-10"
-            iyy="0.0003215"
-            iyz="-1.0165E-10"
-            izz="0.00063022" />
+    <link
+      name="${prefix_}front_right_wheel_link">
+      <inertial>
+        <origin
+          xyz="-1.888E-07 3.5593E-07 0.0069273"
+          rpy="0 0 0" />
+        <mass
+          value="0.13821" />
+        <inertia
+          ixx="0.0003215"
+          ixy="4.0549E-10"
+          ixz="-2.1303E-10"
+          iyy="0.0003215"
+          iyz="-1.0165E-10"
+          izz="0.00063022" />
       </inertial>
       <visual>
@@ -134,5 +144,9 @@
             filename="file://$(find arcs_cohort_description)/meshes/robot1_front_right_wheel_link.STL" />
         </geometry>
-        <material name="yellow"/>
+        <material
+          name="">
+          <color
+            rgba="0.79216 0.81961 0.93333 1" />
+        </material>
       </visual>
       <collision>
@@ -151,5 +165,5 @@
       <origin
         xyz="0.108 -0.089 0.01825"
-        rpy="1.57 0 0" />
+        rpy="1.5708 0 0" />
       <parent
         link="${prefix_}base_link" />
@@ -159,5 +173,117 @@
         xyz="0 0 -1" />
       <dynamics
-        damping="1000000.0"
+        damping="0"
+        friction="0" />
+    </joint>
+    <link
+      name="${prefix_}back_left_wheel_link">
+      <inertial>
+        <origin
+          xyz="-1.888E-07 3.5593E-07 0.0069273"
+          rpy="0 0 0" />
+        <mass
+          value="0.13821" />
+        <inertia
+          ixx="0.0003215"
+          ixy="4.0549E-10"
+          ixz="-2.1303E-10"
+          iyy="0.0003215"
+          iyz="-1.0165E-10"
+          izz="0.00063022" />
+      </inertial>
+      <visual>
+        <origin
+          xyz="0 0 0"
+          rpy="0 0 0" />
+        <geometry>
+          <mesh
+            filename="file://$(find arcs_cohort_description)/meshes/robot1_back_left_wheel_link.STL" />
+        </geometry>
+        <material
+          name="">
+          <color
+            rgba="0.79216 0.81961 0.93333 1" />
+        </material>
+      </visual>
+      <collision>
+        <origin
+          xyz="0 0 0"
+          rpy="0 0 0" />
+        <geometry>
+          <mesh
+            filename="file://$(find arcs_cohort_description)/meshes/robot1_back_left_wheel_link.STL" />
+        </geometry>
+      </collision>
+    </link>
+    <joint
+      name="${prefix_}back_left_wheel_joint"
+      type="continuous">
+      <origin
+        xyz="-0.108 0.089 0.01825"
+        rpy="-1.5708 0 0" />
+      <parent
+        link="${prefix_}base_link" />
+      <child
+        link="${prefix_}back_left_wheel_link" />
+      <axis
+        xyz="0 0 1" />
+      <dynamics
+        damping="0"
+        friction="0" />
+    </joint>
+    <link
+      name="${prefix_}back_right_wheel_link">
+      <inertial>
+        <origin
+          xyz="-1.888E-07 3.5593E-07 0.0069273"
+          rpy="0 0 0" />
+        <mass
+          value="0.13821" />
+        <inertia
+          ixx="0.0003215"
+          ixy="4.0549E-10"
+          ixz="-2.1303E-10"
+          iyy="0.0003215"
+          iyz="-1.0165E-10"
+          izz="0.00063022" />
+      </inertial>
+      <visual>
+        <origin
+          xyz="0 0 0"
+          rpy="0 0 0" />
+        <geometry>
+          <mesh
+            filename="file://$(find arcs_cohort_description)/meshes/robot1_back_right_wheel_link.STL" />
+        </geometry>
+        <material
+          name="">
+          <color
+            rgba="0.79216 0.81961 0.93333 1" />
+        </material>
+      </visual>
+      <collision>
+        <origin
+          xyz="0 0 0"
+          rpy="0 0 0" />
+        <geometry>
+          <mesh
+            filename="file://$(find arcs_cohort_description)/meshes/robot1_back_right_wheel_link.STL" />
+        </geometry>
+      </collision>
+    </link>
+    <joint
+      name="${prefix_}back_right_wheel_joint"
+      type="continuous">
+      <origin
+        xyz="-0.108 -0.089 0.01825"
+        rpy="1.5708 0 0" />
+      <parent
+        link="${prefix_}base_link" />
+      <child
+        link="${prefix_}back_right_wheel_link" />
+      <axis
+        xyz="0 0 -1" />
+      <dynamics
+        damping="0"
         friction="0" />
     </joint>
@@ -202,56 +328,4 @@
       </collision>
     </link>
-    <link
-      name="${prefix_}back_left_wheel_link">
-      <inertial>
-        <origin
-          xyz="-1.888E-07 3.5593E-07 0.0069273"
-          rpy="0 0 0" />
-        <mass
-          value="0.13821" />
-        <inertia
-          ixx="0.0003215"
-          ixy="4.0549E-10"
-          ixz="-2.1303E-10"
-          iyy="0.0003215"
-          iyz="-1.0165E-10"
-          izz="0.00063022" />
-      </inertial>
-      <visual>
-        <origin
-          xyz="0 0 0"
-          rpy="0 0 0" />
-        <geometry>
-          <mesh
-            filename="file://$(find arcs_cohort_description)/meshes/robot1_back_left_wheel_link.STL" />
-        </geometry>
-        <material name="yellow"/>
-      </visual>
-      <collision>
-        <origin
-          xyz="0 0 0"
-          rpy="0 0 0" />
-        <geometry>
-          <mesh
-            filename="file://$(find arcs_cohort_description)/meshes/robot1_back_left_wheel_link.STL" />
-        </geometry>
-      </collision>
-    </link>
-    <joint
-      name="${prefix_}back_left_wheel_joint"
-      type="continuous">
-      <origin
-        xyz="-0.108 0.089 0.01825"
-        rpy="-1.5708 0 0" />
-      <parent
-        link="${prefix_}base_link" />
-      <child
-        link="${prefix_}back_left_wheel_link" />
-      <axis
-        xyz="0 0 1" />
-      <dynamics
-        damping="1000000.0"
-        friction="0" />
-    </joint>
     <joint
       name="${prefix_}camera_mount_joint"
@@ -267,56 +341,4 @@
         xyz="0 0 0" />
     </joint>
-    <link
-      name="${prefix_}back_right_wheel_link">
-      <inertial>
-        <origin
-          xyz="-1.888E-07 3.5593E-07 0.0069273"
-          rpy="0 0 0" />
-        <mass
-          value="0.13821" />
-        <inertia
-          ixx="0.0003215"
-          ixy="4.0549E-10"
-          ixz="-2.1303E-10"
-          iyy="0.0003215"
-          iyz="-1.0165E-10"
-          izz="0.00063022" />
-      </inertial>
-      <visual>
-        <origin
-          xyz="0 0 0"
-          rpy="0 0 0" />
-        <geometry>
-          <mesh
-            filename="file://$(find arcs_cohort_description)/meshes/robot1_back_right_wheel_link.STL" />
-        </geometry>
-        <material name="yellow"/>
-      </visual>
-      <collision>
-        <origin
-          xyz="0 0 0"
-          rpy="0 0 0" />
-        <geometry>
-          <mesh
-            filename="file://$(find arcs_cohort_description)/meshes/robot1_back_right_wheel_link.STL" />
-        </geometry>
-      </collision>
-    </link>
-    <joint
-      name="${prefix_}back_right_wheel_joint"
-      type="continuous">
-      <origin
-        xyz="-0.108 -0.089 0.01825"
-        rpy="1.5708 0 0" />
-      <parent
-        link="${prefix_}base_link" />
-      <child
-        link="${prefix_}back_right_wheel_link" />
-      <axis
-        xyz="0 0 -1" />
-      <dynamics
-        damping="1000000.0"
-        friction="0" />
-    </joint>
-    </xacro:macro>
+  </xacro:macro>
 </robot>
