Commit message: Add rover usd model

File: description/robot2.urdf (robot description, URDF)
Before this commit: robot None, 0 links, 0 joints
Links:
- added link back_left_wheel_link, mass 0.13821; collision mesh filename=file:///home/cohort/cohort_ws/install/arcs_cohort_descripti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; visual mesh filename=file:///home/cohort/cohort_ws/install/arcs_cohort_descripti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
- added link back_right_wheel_link, mass 0.13821; collision mesh filename=file:///home/cohort/cohort_ws/install/arcs_cohort_descripti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; visual mesh filename=file:///home/cohort/cohort_ws/install/arcs_cohort_descripti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
- added link base_footprint
- added link base_link, mass 0.629688250105366; collision mesh filename=file:///home/cohort/cohort_ws/install/arcs_cohort_descripti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; visual mesh filename=file:///home/cohort/cohort_ws/install/arcs_cohort_descripti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
- added link front_left_wheel_link, mass 0.13821; collision mesh filename=file:///home/cohort/cohort_ws/install/arcs_cohort_descripti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; visual mesh filename=file:///home/cohort/cohort_ws/install/arcs_cohort_descripti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
- added link front_right_wheel_link, mass 0.13821; collision mesh filename=file:///home/cohort/cohort_ws/install/arcs_cohort_descripti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; visual mesh filename=file:///home/cohort/cohort_ws/install/arcs_cohort_descripti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
- added link zedm_camera_center; collision mesh filename=file:///opt/ros/jazzy/share/zed_msgs/meshes/zedm.stl; visual mesh filename=file:///opt/ros/jazzy/share/zed_msgs/meshes/zedm.stl
- added link zedm_camera_link
- added link zedm_camera_mount_link, mass 0; collision mesh filename=file:///home/cohort/cohort_ws/install/arcs_cohort_descripti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; visual mesh filename=file:///home/cohort/cohort_ws/install/arcs_cohort_descripti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
- added link zedm_left_camera_frame
- added link zedm_left_camera_optical_frame
- added link zedm_right_camera_frame
- added link zedm_right_camera_optical_frame
Joints:
- added joint back_left_wheel_joint: type continuous, parent base_link, child back_left_wheel_link, origin xyz=-0.108 0.089 0.01825 rpy=-1.5708 0 0, axis 0 0 1
- added joint back_right_wheel_joint: type continuous, parent base_link, child back_right_wheel_link, origin xyz=-0.108 -0.089 0.01825 rpy=1.5708 0 0, axis 0 0 -1
- added joint base_joint: type fixed, parent base_footprint, child base_link, origin xyz=0.12 0.0 0.0 rpy=0 0 0
- added joint camera_mount_joint: type fixed, parent base_link, child zedm_camera_mount_link, origin xyz=0.1345 0.0036809 0.039145 rpy=0 0 0, axis 0 0 0
- added joint front_left_wheel_joint: type continuous, parent base_link, child front_left_wheel_link, origin xyz=0.108 0.089 0.01825 rpy=-1.57 0 0, axis 0 0 1
- added joint front_right_wheel_joint: type continuous, parent base_link, child front_right_wheel_link, origin xyz=0.108 -0.089 0.01825 rpy=1.57 0 0, axis 0 0 -1
- added joint zedm_camera_center_joint: type fixed, parent zedm_camera_link, child zedm_camera_center, origin xyz=0 0 0.01325 rpy=0 0.0 0
- added joint zedm_camera_mount_to_camera: type fixed, parent zedm_camera_mount_link, child zedm_camera_link, origin xyz=0.015 -0.0068 0 rpy=0 0 0
- added joint zedm_left_camera_joint: type fixed, parent zedm_camera_center, child zedm_left_camera_frame, origin xyz=0.0 0.0315 0 rpy=0 0 0
- added joint zedm_left_camera_optical_joint: type fixed, parent zedm_left_camera_frame, child zedm_left_camera_optical_frame, origin xyz=0 0 0 rpy=-1.5707963267948966 0.0 -1.5707963267948966
- added joint zedm_right_camera_joint: type fixed, parent zedm_camera_center, child zedm_right_camera_frame, origin xyz=0.0 -0.0315 0 rpy=0 0 0
- added joint zedm_right_camera_optical_joint: type fixed, parent zedm_right_camera_frame, child zedm_right_camera_optical_frame, origin xyz=0 0 0 rpy=-1.5707963267948966 0.0 -1.5707963267948966
